Commit message: 完成关节空间和笛卡尔空间任务，完成 ros2_control 具体链路。 问题：机械臂抖动和joint1扭动

File: kdl/src/model/robotic_arm.urdf (robot description, URDF)
Before this commit: robot robotic_arm, 8 links, 7 joints
Links:
- link base_link: geometry collision mesh filename=package://kdl_tools/model/base_link.STL; visual mesh filename=package://kdl_tools/model/base_link.STL
- link link1: geometry collision mesh filename=package://kdl_tools/model/link1.STL; visual mesh filename=package://kdl_tools/model/link1.STL
- link link2: geometry collision mesh filename=package://kdl_tools/model/link2.STL; visual mesh filename=package://kdl_tools/model/link2.STL
- link link3: geometry collision mesh filename=package://kdl_tools/model/link3.STL; visual mesh filename=package://kdl_tools/model/link3.STL
- link link4: geometry collision mesh filename=package://kdl_tools/model/link4.STL; visual mesh filename=package://kdl_tools/model/link4.STL
- link link5: geometry collision mesh filename=package://kdl_tools/model/link5.STL; visual mesh filename=package://kdl_tools/model/link5.STL
- link link6: geometry collision mesh filename=package://kdl_tools/model/link6.STL; visual mesh filename=package://kdl_tools/model/link6.STL

Commit message: 从 6 轴臂迁移到 4 轴臂：模型替换、控制栈适配、PID 重新整定、文档同步
本次把项目里的机器人从 6 轴整体换成 4 轴，并把因此失效的控制链路全部修复到可运行、
可跟踪的状态。下面是完成的内容、实测证据，以及尚未解决的问题。

════════════════════════════════════════════════════════════════════
一、模型替换：6 轴 → 4 轴
════════════════════════════════════════════════════════════════════
* src/model/ 整体替换：link1..link4（删除 link5.STL / link6.STL），
  URDF / MJCF / scene / CSV 全部更新。
* 新 URDF 的差异（相对旧模型）：
  - 没有 world link 与 world_to_base，base_link 直接成为根 link；
  - 四个关节 <limit effort> 均为 50 N·m（旧臂是 50/50/50/100/50/50）；
  - 行程变化很大：joint1 ±3.14→±1.57，joint2 ±1.57→±3.0，
    joint3 ±2.8→±3.14，joint4 -1.82..1.92→±1.57；
  - 完全没有 <dynamics>（旧 joint6 有 damping/friction）。
* 按 src/model 既有的书写规则生成 4 个 MJCF：
  robotic_arm.xml（位置伺服）、robotic_arm_torque.xml（纯力矩）、
  scene.xml、scene_torque.xml。
  - 姿态一律用 quat="w x y z"，由 URDF rpy 按 Rz(yaw)·Ry(pitch)·Rx(roll) 换算；
    该换算实现先用旧模型的 URDF→MJCF 已有数据反验（最大偏差 4.6e-13）再用于新模型。
  - fullinertia 按 MuJoCo 的 Ixx Iyy Izz Ixy Ixz Iyz 顺序重排，并逐项校验
    张量正定且满足三角不等式（MuJoCo 加载时会强校验）。
  - 力矩版排除全部 10 对连杆自碰撞（覆盖 5 个 body 的所有组合），
    位置版只排除相邻 4 对 —— 与旧模型的做法保持一致。

════════════════════════════════════════════════════════════════════
二、控制栈从 6 轴假设适配到 4 轴
════════════════════════════════════════════════════════════════════
* kdl_tools.hpp：kDefaultTipLink "link6" → "link4"（含相关文档注释）。
* kdl_task_router.hpp：同一默认值的**第二份硬编码副本**。该头文件为了不把
  <urdf/model.h> 带进公共头而自行写了字面量，所以只改 kDefaultTipLink 治不到它，
  实测表现为控制节点与 control_demo 仍然建链失败。
* robotic_arm_mujoco.urdf.xacro：删除 joint5/joint6 的 <xacro:arm_joint>。
* controllers.yaml / kdl_control_node.cpp / kdl_identify_node.cpp：
  joints / joint_names 从 6 个改为 4 个。
* mujoco_pids.yaml：删除 joint5/joint6；joint4 的 u_clamp ±100 → ±50（对齐 URDF effort）。
* 重建后清掉 install/ 里残留的 link5.STL / link6.STL
  （install(DIRECTORY) 只覆盖不删除，会留下幽灵文件）。

════════════════════════════════════════════════════════════════════
三、PID 增益按新臂重新整定（本次的核心工作）
════════════════════════════════════════════════════════════════════
直接沿用旧臂增益会让 joint3 自激：实测关节速度在 ±40~70 rad/s 之间抖振
（URDF 速度上限只有 10），轨迹终点残差 1.34 rad，控制器完全无法跟踪。

整定分两步，中间纠正过一次判断：

1) 先按 kp = J·ωn²、kd = 2ζ·J·ωn（ωn=15, ζ=1）重算。
   各关节的等效惯量 = 该关节所有远端连杆绕该关节轴的复合刚体惯量
   （用 URDF/MJCF 的质量、惯量、质心逐段复合算出）。
   算法可信度：旧臂 joint2 算得 1.4755 kg·m²，与《力矩控制问题报告》独立实测的
   ≈1.4 kg·m² 吻合。
   → 稳定性解决（抖振归零），但 joint3 变得极慢，轨迹仍然失败。

2) 发现真正的判据不是带宽而是**柔度 τ_g/kp**（前馈残差会放大成多大的稳态误差）。
   实测各关节稳态保持力矩后：

     关节     τ_g        kp         τ_g/kp
     joint1   4.666     80.29      0.058 rad
     joint2   2.013     18.62      0.108 rad
     joint3   0.093     0.0529     1.76 rad   ← 唯一的异常
     joint4   0.0033    0.3553     0.009 rad

   joint3 的 J 极小，J·ωn² 给出的绝对刚度（0.053 N·m/rad）比它要抵抗的重力负载
   （0.093 N·m）还小 —— 重力扰动不随 J 缩小，所以该规则对小惯量关节失效。
   按"把柔度压到与其它关节同量级（~0.05 rad）"反推：kp ≈ τ_g/0.05 ≈ 1.9。

最终增益（config/mujoco_pids.yaml，文件头部有完整推导注释）：
     joint1  p=80.29   d=10.71
     joint2  p=18.62   d=2.483
     joint3  p=1.9     d=0.078
     joint4  p=0.3553  d=0.04738

════════════════════════════════════════════════════════════════════
四、文档同步
════════════════════════════════════════════════════════════════════
* README.md：关节映射表（6→4 行，joint4 的 ctrlrange ±100→±50）、
  joints/joint_names/max_acceleration 默认值、启动日志摘录、服务调用示例、
  两处"实测"表换成本次的真实数据。
* PLAN_TORQUE.md：MJCF <actuator> 片段、controllers.yaml 示例、joint_names、
  事实表 F2/F6（旧 kp 值与已失效的行号）、风险表把"模型差异"标为**已发生**
  并记录实际后果、计划vs实际表的增益/阻尼/接触三行。
* 力矩控制问题报告.md：**只加注、不改写**。该文记录的是旧 6 轴臂的真实实测，
  改写等于伪造历史，所以在顶部插入历史说明，逐条点明哪些是旧臂事实、
  哪些结论仍适用（问题 1/5）、哪些必须重做（问题 2 的 PID 重调）。
* PLAN.md：顶部本就有"已被 PLAN_TORQUE.md 取代，仅作历史记录保留"的横幅，未改。
* 代码注释 9 处：build_from_urdf.cpp、control_demo.cpp、vel_acc_demo.cpp、
  quintic_demo.cpp、kdl_tools_print.hpp、kdl_identify_node.cpp、
  regressor_lsq_demo.cpp、plot_quintic.py。

════════════════════════════════════════════════════════════════════
五、其他
════════════════════════════════════════════════════════════════════
* regressor_lsq_demo：新增"[7] 结构性不可辨识的参数"分析 —— 用回归列范数把
  "解析上与 τ 无关"和"辨识不出来"区分开。
* 新增 demo 输出：cartesian_trajectory.csv、quintic_trajectory.csv。

════════════════════════════════════════════════════════════════════
实测结果
════════════════════════════════════════════════════════════════════
* colcon build --packages-select kdl_tools → exit 0。
* 端到端 ros2 launch arm_mujoco_control_with_bridge.launch.py（含 GUI）：
  MuJoCo 加载 scene_torque.xml → 注册 joint1..joint4 四个执行器 →
  硬件接口 arm_hw 加载 → joint_state_broadcaster 与 kdl_effort_controller 均
  Configured and activated，无任何报错。
* 关节空间任务（service /control_task）：
    [1.0,-1.0,1.2,0.8]  (起 [0.87,2.40,0.30,0.96])  自动 6.50 s → error_code=0
    [0.0,0.8,0.0,1.4]                               自动 3.44 s → error_code=0
    [1.2,-1.2,1.4,0.6]                              自动 3.83 s → error_code=0
  四轴终点残差全部 0.0000 rad，过冲为 0，静止后速度 5e-14 rad/s。
* 迁移前后对比（同一目标轨迹）：
    旧增益 p=70     → error 8，joint3 残差 1.344 rad，max|q̇| 40.3 rad/s
    仅按 J 缩放     → error 8，joint3 残差 1.174 rad
    修正后 p=1.9    → error 0，joint3 残差 0.0000 rad

════════════════════════════════════════════════════════════════════
项目当前存在的问题（本次未解决）
════════════════════════════════════════════════════════════════════
[1] 大行程轨迹在**峰值速度段**出现 0.1~0.2 s 的高频振荡，四轴同时反向，
    实测关节速度冲到 14~22 rad/s（URDF 上限 10）。7 次实测出现 5 次，
    幅度小的回程那次完全没有。自恢复、不影响最终精度（最近一次过冲为 0），
    但根因未定位 —— 控制器日志无告警，/kdl_effort_controller/status 正常。

[2] u_clamp 与 URDF <limit effort> 都是 ±50 N·m，对 joint3 不物理：
    该连杆仅 82 g、等效惯量 2.35e-4 kg·m²，50 N·m 对应 2e6 rad/s²。
    现在增益低所以打不到限幅，但这等于**没有力矩保护**，真机上有风险。
    需要按真实电机能力重设，且要同步改 URDF、两个 MJCF、mujoco_pids.yaml 四处。

[3] 控制器被 spawner 激活之前（约 0.5 s）effort 恒为 0，机械臂在重力下
    **自由下落**，落到随机位姿才被接住。这是旧报告 §3 就记录的既有问题，
    4 轴臂上更明显（joint2 行程从 ±1.57 扩到 ±3.0，下落幅度更大），
    且新模型没有关节阻尼来缓解。

[4] 两个示例仍然损坏：
    - vel_acc_demo：KDL 的 ChainIkSolverVel_wdls 对 4 关节链触发 Eigen 断言
      （Block 维度越界）。**不在控制路径上**，只有该 demo 与两个库函数用它。
    - control_demo：q_start/q_goal 与 max_acceleration 仍是 6 元素硬编码，
      与 4 关节链不匹配，在校验处失败。

[5] 新 URDF 没有 world link，带惯量的 base_link 成了根，KDL 会丢弃根连杆惯量
    并打印 WARN。固定基座下功能无害，想消掉就照旧模型加无质量 world + fixed joint。

[6] kdl_control_node.cpp 的 (n == 6) 默认加速度分支已成死代码，
    4 轴走 else（全部 30 rad/s²），该组值未按新臂整定。

[7] 参数辨识链路从未跑过。draw/identification_params.csv 仍是旧 6 轴产物
    （49 行，含 link5/link6/joint5/joint6），索引编号对应 6 轴参数集。
    激励轨迹优化器会读 URDF 限位自适应、不会越界，但 joint1/joint4 行程缩小
    后激励空间变小、可辨识性下降。

[8] 笛卡尔任务：4 自由度张不满 6 维任务空间，kdl_cartesian_space_task 会
    静默给出最小二乘解。未实测。

File: kdl/src/model/robotic_arm.urdf (robot description, URDF)
Before this commit: robot robotic_arm, 8 links, 7 joints
Links:
- removed link link5
- removed link link6
- removed link world
- link base_link: mass 0.905716018714615 -> 0.446116144380579
- link link1: mass 1.91180538368796 -> 0.43178795433662
- link link2: mass 1.09233144358037 -> 0.334546886253206
- link link3: mass 0.750870225721497 -> 0.0818036914981158
- link link4: mass 0.328855136025888 -> 0.269974503355347
Joints:
- removed joint joint5
- removed joint joint6
- removed joint world_to_base
- joint joint1: limit lower=-3.14 upper=3.14 effort=50 velocity=10 -> lower=-1.57 upper=1.57 effort=50 velocity=10; origin xyz=6.34132927793407E-05 -0.00167405073291106 0.0278500000000087 rpy=0 0 0 -> xyz=0 -0.04 0.05 rpy=1.5708 -1.57 -3.1416
- joint joint2: axis 0 0 -1 -> 0 -1 0; limit lower=-1.57 upper=1.57 effort=50 velocity=10 -> lower=-3.0 upper=3.0 effort=50 velocity=10; origin xyz=0.00565491862295636 0.0185517283813911 0.0710733482199691 rpy=-1.5707963267949 -1.5708 0 -> xyz=0.374 0 0.0401 rpy=1.5708 0.0 0.0
- joint joint3: axis 0 0 -1 -> 0 0 1; limit lower=-2.8 upper=2.8 effort=50 velocity=10 -> lower=-3.14 upper=3.14 effort=50 velocity=10; origin xyz=0.500001547205985 -0.00750000000003981 0.0418960557056171 rpy=3.14159265358979 0 0 -> xyz=0.3384 -0.0055 0.045 rpy=-1.5708 -1.5708 -1.5708
- joint joint4: axis 0 0 -1 -> 0 0 1; limit lower=-1.82 upper=1.92 effort=100 velocity=1 -> lower=-1.57 upper=1.57 effort=50 velocity=10; origin xyz=0.493372719987381 -0.000717203264851807 -0.0115 rpy=3.14159265358979 0 1.5708 -> xyz=0.00079568 0.018983 0.043 rpy=-1.5708 -1.5708 3.14

File: kdl/src/ros2_control/urdf/robotic_arm_mujoco.urdf.xacro (robot description, xacro)
@@ -13,6 +13,6 @@
     控制器 ──> command_interface(关节力矩) ──> MuJoCo ctrl（<motor> 直接当力矩施加）
   对应关系速查：
-    关节      joint1..joint6        （URDF，也是 MJCF 里的 joint 名）
-    执行器    motor1..motor6        （MJCF <motor .../>，ctrl = 关节力矩 [N·m]）
+    关节      joint1..joint4        （URDF，也是 MJCF 里的 joint 名）
+    执行器    motor1..motor4        （MJCF <motor .../>，ctrl = 关节力矩 [N·m]）
     传动      1:1 直连，不需要 <transmission>（详见文件末尾注释与 README）
   力矩控制的两个硬前提（改这里时别忘）：
@@ -59,5 +59,5 @@
            <param name="odom_topic">/simulator/floating_base_state</param> -->
     </hardware>
-    <!-- 关节 ↔ 接口声明。六个关节接口完全相同，用宏展开避免手抄六遍。 -->
+    <!-- 关节 ↔ 接口声明。四个关节接口完全相同，用宏展开避免手抄四遍。 -->
     <xacro:macro name="arm_joint" params="name">
       <joint name="${name}">
@@ -81,6 +81,4 @@
     <xacro:arm_joint name="joint3"/>
     <xacro:arm_joint name="joint4"/>
-    <xacro:arm_joint name="joint5"/>
-    <xacro:arm_joint name="joint6"/>
     <!-- ===================== 传动（transmission）配置说明 =====================
          当前的 1:1 直连不需要任何 <transmission>：

Commit message: 放宽关节限位：joint1/joint4 补足到 ±1.5708，joint2 放宽到 ±3.1
## 改动
                    改前        改后
    joint1          ±1.57      ±1.5708     （补足到精确的 π/2）
    joint2          ±3.0       ±3.1        （放宽 0.1 rad ≈ 5.7°）
    joint3          ±3.14      ±3.14       （不动）
    joint4          ±1.57      ±1.5708     （补足到精确的 π/2）

## 为什么必须同时改三处
限位有三个独立来源，只改一处不起作用：

| 来源 | 谁读 | 改不改 |
|---|---|---|
| URDF `<limit lower upper>` | KDL 链 → RobotContext.q_min/q_max | **改** |
| MJCF `<joint range>` | MuJoCo 物理 | **改**（真正把关节卡死的是它） |
| MJCF 执行器 `ctrlrange` | MuJoCo 执行器 | position 版要跟着改；torque 版的 ±50 是力矩，不动 |

只改 URDF 的后果是：任务层放行 → 控制器往限位外输出 → MuJoCo 照旧夹住 →
控制器对着夹持较劲。所以三个文件一起改：
  src/model/robotic_arm.urdf              4 处 <limit>
  src/model/robotic_arm_torque.xml        3 处 <joint range>（力矩版，launch 实际用这一份）
  src/model/robotic_arm.xml               3 处 <joint range> + 3 处 <position ctrlrange>
                                          （position 版，作为回退保留，也一并对齐）
scene.xml / scene_torque.xml 只 include 本体文件，没有自己的 range，不用改。

## 顺带
PLAN_TORQUE.md 里"joint2 行程为 ±3.0"改为 ±3.1。

## 验证
- 已安装副本确认生效（install/kdl_tools/share/kdl_tools/model/ 下三个文件都是新值）
- 服务端到端：`joint2 = 3.15` 被拒并报出新行程 —— 证明 URDF 限位确实被动态加载：
    "第 2 个关节的目标 3.15 rad 超出行程 [-3.1, 3.1] rad"
- 7 个 demo 全部 exit 0
- 仿真：归位 + 笛卡尔任务均 success，末态关节角
  [0.499999, -0.399999, 0.600046, 0.300002]

## 实测没有达到预期的部分（如实记录）
改这个的动机之一是缓解 B4（控制器激活前自由下落撞在限位上）。**实测无效**：
臂仍然每次启动都自由落体并卡在限位上（甚至 joint2/joint3 因为行程更宽而越界更多）。
重跑多次观察到的落地姿态在"卡在限位"与"自然悬停"之间跳变，说明落地本身是混沌的，
一次观察不足以说明问题 —— 不能拿单次样本当作"放宽限位让臂不再卡死"的证据。

真正要解决 B4 得给 MJCF 加关节阻尼，或让控制器先于自由落体接管，本次未做。

## 侧记
放宽之后暴露出限位校验容差过紧的问题（原值 1e-3，而实测越界可达 9.3e-3），
会在第 0 个采样点拒掉机器人自己的当前状态。下一个提交单独修。

File: kdl/src/model/robotic_arm.urdf (robot description, URDF)
Before this commit: robot robotic_arm, 6 links, 5 joints
Joints:
- joint joint1: limit lower=-1.57 upper=1.57 effort=50 velocity=10 -> lower=-1.5708 upper=1.5708 effort=50 velocity=10
- joint joint2: limit lower=-3.0 upper=3.0 effort=50 velocity=10 -> lower=-3.1 upper=3.1 effort=50 velocity=10
- joint joint4: limit lower=-1.57 upper=1.57 effort=50 velocity=10 -> lower=-1.5708 upper=1.5708 effort=50 velocity=10
